Commit message: Added transparent sphere to grip target for better visualization

File: robotic_stacking/resources/KinovaG3_7DOF_HandEgrip.urdf (robot description, URDF)
Before this commit: robot KinovaG3_7DOF_HandEgrip, 12 links, 11 joints
Links:
- link gripper_target: geometry visual sphere radius=0.025

Commit message: Changed orientation of target link joint to keep gripper facing downward

File: robotic_stacking/resources/KinovaG3_7DOF_HandEgrip.urdf (robot description, URDF)
Before this commit: robot KinovaG3_7DOF_HandEgrip, 12 links, 11 joints
Joints:
- joint target_to_gripper: origin xyz=0 0 0.125 rpy=0 0 0 -> xyz=0 0 0.125 rpy=0 3.14159265 0
